File: theremin.kicad_pcb (KiCad board)
At the start: 2 copper layers, 102 parts, among them J1 Audio Out, J2 12VAC, Q1 2N3904, Q2 2N3904, Q3 2N3904, Q4 2N3904, Q5 2N3904, Q6 2N3904, Q7 2N3904, Q8 2N3904, U1 LM13600, U2 L7812, U3 L7912

Commit message: Initial placement for pcb.
Parts:
- R14: moved to B.Cu
- moved J1 136.8 mm to (168.2, 172.4)
- moved RV1 136.0 mm to (136.6, 172.4), turned to -90 degrees
- moved L1 129.2 mm to (241.3, 46.4)
- moved L2 129.2 mm to (241.3, 51.3)
- moved L3 129.2 mm to (241.3, 56.1)
- moved L4 129.2 mm to (241.3, 61.0)
- moved R3 127.5 mm to (271.8, 114.3), turned to 90 degrees
- moved R1 127.2 mm to (266.7, 114.3), turned to 90 degrees
- moved AE2 121.9 mm to (246.4, 30.5)
- moved R2 120.7 mm to (261.6, 114.3), turned to 90 degrees
- moved RV2 118.4 mm to (122.5, 172.4), turned to -90 degrees
- moved L5 117.2 mm to (266.7, 83.8)
- moved C4 116.6 mm to (279.4, 121.9)
- moved C8 116.5 mm to (109.2, 147.3)
- moved R4 112.2 mm to (256.5, 114.3), turned to 90 degrees
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Connections:
- R14 pad 1: Net-(D1-A) -> (no net)
- R14 pad 2: Volume Antenna A -> (no net)

Commit message: Placed in smd and through.
Parts:
- added D6: LED, Connector_PinHeader_2.54mm:PinHeader_1x02_P2.54mm_Vertical, F.Cu at (53.3, 56.0)
- added R41: R_US, Resistor_SMD:R_0805_2012Metric, F.Cu at (43.0, 57.8)
- added REF**: MountingHole_2.1mm, MountingHole:MountingHole_2.1mm, F.Cu at (40.9, 43.4)
- added REF**: MountingHole_2.1mm, MountingHole:MountingHole_2.1mm, F.Cu at (149.6, 46.0)
- added REF**: MountingHole_2.1mm, MountingHole:MountingHole_2.1mm, F.Cu at (149.4, 28.2)
- added REF**: MountingHole_2.1mm, MountingHole:MountingHole_2.1mm, F.Cu at (41.4, 28.2)
- added SW1: SW_SPDT, Button_Switch_THT:SW_SPST_Omron_B3F-315x_Angled, F.Cu at (45.5, 61.9)
- AE1, AE2: footprint Connector_Coaxial:BNC_Amphenol_031-5539_Vertical -> Connector_Pin:Pin_D1.3mm_L11.0mm
- C1, C12, C14, C15, C16, C2, C24, C26, C3, C5, C6, C7, C9: footprint Capacitor_THT:C_Disc_D11.0mm_W5.0mm_P7.50mm -> Capacitor_SMD:C_0805_2012Metric
- C10, C11, C13, C17, C18, C25, C4, C8: footprint Capacitor_THT:CP_Radial_D10.0mm_P3.80mm -> Capacitor_THT:CP_Radial_D5.0mm_P2.50mm
- C19, C20: footprint Capacitor_THT:CP_Radial_D10.0mm_P3.80mm -> Capacitor_THT:CP_Radial_D10.0mm_P3.50mm
- C21, C22, C23, C27: footprint Capacitor_THT:C_Disc_D11.0mm_W5.0mm_P7.50mm -> Capacitor_SMD:C_1812_4532Metric
- D1, D4, D5: footprint Diode_THT:D_DO-35_SOD27_P7.62mm_Horizontal -> Diode_SMD:D_2010_5025Metric
- D2, D3: footprint Diode_THT:D_DO-41_SOD81_P10.16mm_Horizontal -> Diode_SMD:D_2010_5025Metric
- L1, L10, L11, L2, L3, L4, L5, L6, L7, L8, L9: footprint Inductor_THT:L_Axial_L7.0mm_D3.3mm_P12.70mm_Horizontal_Fastron_MICC -> Inductor_SMD:L_1210_3225Metric
- R1, R10, R11, R12, R13, R15, R16, R17, R18, R19, R2, R20, R21, R22, R23, R24, R25, R26, R27, R28, R29, R3, R30, R31, R32, R33, R34, R35, R36, R37, R38, R39, R4, R40, R5, R6, R7, R8, R9: footprint Resistor_THT:R_Axial_DIN0207_L6.3mm_D2.5mm_P10.16mm_Horizontal -> Resistor_SMD:R_0805_2012Metric
- R14: footprint Resistor_THT:R_Axial_DIN0207_L6.3mm_D2.5mm_P10.16mm_Horizontal -> Resistor_SMD:R_0805_2012Metric; moved to F.Cu
- moved C4 167.5 mm to (141.0, 27.7), turned to -90 degrees
- moved R3 150.2 mm to (138.8, 44.5), turned to 0 degrees
- moved C3 148.0 mm to (139.0, 47.8), turned to 180 degrees
- moved R1 146.9 mm to (139.2, 41.4), turned to 180 degrees
- moved R2 144.5 mm to (139.2, 37.6), turned to 180 degrees
- moved R4 142.3 mm to (139.2, 33.8), turned to 180 degrees
- moved C1 131.9 mm to (145.5, 45.9), turned to 90 degrees
- moved Q1 131.3 mm to (143.0, 40.1), turned to -90 degrees
- moved R34 129.5 mm to (133.6, 43.8), turned to 180 degrees
- moved L5 129.2 mm to (143.0, 46.4), turned to -90 degrees
- moved Q2 126.2 mm to (143.0, 33.8), turned to -90 degrees
- moved C25 122.8 mm to (125.7, 27.7)
- moved RV4 120.9 mm to (133.9, 58.2)
- moved RV2 118.6 mm to (91.7, 57.9)
- moved RV1 118.3 mm to (105.7, 58.2)
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Connections:
- J2 pad 1: VAC -> Net-(SW1-C)
- R14 pad 1: (no net) -> Net-(D1-A)
- R14 pad 2: (no net) -> Volume Antenna A
Routing:
- added copper zone on B.Cu, net Earth
- added copper zone on F.Cu, net Earth
Other:
- board outline added: 139.7 x 38.1 mm
