File: theremin.kicad_pcb (KiCad board)
At the start: 2 copper layers, 139.7 x 38.1 mm, 108 parts, among them J1 Audio Out, J2 12VAC, Q1 2N3904, Q2 2N3904, Q3 2N3904, Q4 2N3904, Q5 2N3904, Q6 2N3904, Q7 2N3904, Q8 2N3904, SW1 SW_SPDT, U1 LM13600, U2 L7812, U3 L7912

Commit message: Finished VPO
Parts:
- C1, C12, C14, C15, C16, C2, C24, C26, C3, C5, C6, C7, C9: footprint Capacitor_SMD:C_0805_2012Metric -> Capacitor_THT:C_Disc_D3.0mm_W1.6mm_P2.50mm
- C21, C22, C23, C27: footprint Capacitor_SMD:C_1812_4532Metric -> Capacitor_THT:C_Disc_D3.8mm_W2.6mm_P2.50mm
- D1, D2, D3, D4, D5: footprint Diode_SMD:D_2010_5025Metric -> Diode_THT:D_DO-35_SOD27_P7.62mm_Horizontal
- L1, L10, L11, L2, L3, L4, L5, L6, L7, L8, L9: footprint Inductor_SMD:L_1210_3225Metric -> Inductor_THT:L_Axial_L5.3mm_D2.2mm_P7.62mm_Horizontal_Vishay_IM-1
- R1, R10, R11, R12, R13, R14, R15, R16, R17, R18, R19, R2, R20, R21, R22, R23, R24, R25, R26, R27, R28, R29, R3, R30, R31, R32, R33, R34, R35, R36, R37, R38, R39, R4, R40, R41, R5, R6, R7, R8, R9: footprint Resistor_SMD:R_0805_2012Metric -> Resistor_THT:R_Axial_DIN0204_L3.6mm_D1.6mm_P5.08mm_Horizontal
- moved C2 42.0 mm to (140.0, 49.2), turned to 90 degrees
- moved REF** 14.9 mm to (40.6, 28.6)
- moved L5 14.7 mm to (149.9, 32.0), turned to -90 degrees
- moved R2 14.1 mm to (147.3, 46.7)
- moved R6 12.3 mm to (68.3, 35.8), turned to -90 degrees
- moved R8 12.0 mm to (70.6, 42.6)
- moved C10 9.87 mm to (92.5, 43.1), turned to 90 degrees
- moved R39 9.74 mm to (86.9, 29.1), turned to 0 degrees
- moved R7 9.35 mm to (75.4, 40.3)
- moved R9 9.29 mm to (86.9, 31.7), turned to 0 degrees
- moved C23 9.08 mm to (110.7, 44.5)
- moved C9 8.74 mm to (81.0, 37.2)
- moved C7 8.09 mm to (75.9, 35.3)
- moved C11 7.74 mm to (91.2, 36.0)
- moved C4 7.69 mm to (144.3, 30.9)
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Routing:
- net +12V: track 98.9 -> 37.3 mm, vias 1 -> 0
- net Volume Tuning: track 0.00 -> 39.8 mm
- net Net-(Q3-C): track 20.9 -> 46.0 mm
- net -12V: track 47.7 -> 24.3 mm, vias 2 -> 0
- net Volume Antenna B: track 5.13 -> 26.7 mm
- net Net-(R29-Pad1): track 17.0 -> 0.00 mm
- net Net-(D5-K): track 17.0 -> 0.11 mm
- net Net-(C24-Pad1): track 12.1 -> 0.00 mm
- net Volume Antenna A: track 23.9 -> 14.2 mm
- net Net-(U1C--): track 9.43 -> 0.00 mm
- net Net-(D5-A): track 9.41 -> 0.00 mm
- net Audio Out: track 8.09 -> 0.00 mm
- net Detector: track 0.00 -> 7.89 mm
- net Net-(C25-Pad2): track 7.75 -> 0.00 mm
- net PitchAntenna: track 9.75 -> 17.0 mm
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