File: vca.kicad_sch (KiCad schematic)
At the start: 24 parts, among them U1 LM13600

Commit message: Placed in smd and through.
Parts:
- C23, C27: footprint Capacitor_THT:C_Disc_D11.0mm_W5.0mm_P7.50mm -> Capacitor_SMD:C_1812_4532Metric
- C24, C26: footprint Capacitor_THT:C_Disc_D11.0mm_W5.0mm_P7.50mm -> Capacitor_SMD:C_0805_2012Metric
- C25: footprint Capacitor_THT:CP_Radial_D10.0mm_P3.80mm -> Capacitor_THT:CP_Radial_D5.0mm_P2.50mm
- D4, D5: footprint Diode_THT:D_DO-35_SOD27_P7.62mm_Horizontal -> Diode_SMD:D_2010_5025Metric
- R23, R24, R25, R26, R27, R28, R29, R30, R31, R32, R33, R34, R35, R36, R37, R38: footprint Resistor_THT:R_Axial_DIN0207_L6.3mm_D2.5mm_P10.16mm_Horizontal -> Resistor_SMD:R_0805_2012Metric
Changed lines of the file:
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@@
       (effects (font (size 1.27 1.27)) (justify left))
     )
-    (property "Footprint" "Resistor_THT:R_Axial_DIN0207_L6.3mm_D2.5mm_P10.16mm_Horizontal" (at 114.046 100.584 90)
+    (property "Footprint" "Resistor_SMD:R_0805_2012Metric" (at 114.046 100.584 90)
       (effects (font (size 1.27 1.27)) hide)
     )
@@
       (effects (font (size 1.27 1.27)))
     )
-    (property "Footprint" "Resistor_THT:R_Axial_DIN0207_L6.3mm_D2.5mm_P10.16mm_Horizontal" (at 84.836 64.516 90)
+    (property "Footprint" "Resistor_SMD:R_0805_2012Metric" (at 84.836 64.516 90)
       (effects (font (size 1.27 1.27)) hide)
     )
@@
       (effects (font (size 1.27 1.27)))
     )
-    (property "Footprint" "Resistor_THT:R_Axial_DIN0207_L6.3mm_D2.5mm_P10.16mm_Horizontal" (at 147.574 95.504 90)
+    (property "Footprint" "Resistor_SMD:R_0805_2012Metric" (at 147.574 95.504 90)
       (effects (font (size 1.27 1.27)) hide)
     )
@@
       (effects (font (size 1.27 1.27)))
     )
-    (property "Footprint" "Resistor_THT:R_Axial_DIN0207_L6.3mm_D2.5mm_P10.16mm_Horizontal" (at 87.376 105.156 90)
+    (property "Footprint" "Resistor_SMD:R_0805_2012Metric" (at 87.376 105.156 90)
       (effects (font (size 1.27 1.27)) hide)
     )
@@
       (effects (font (size 1.27 1.27)) (justify left))
     )
-    (property "Footprint" "Capacitor_THT:C_Disc_D11.0mm_W5.0mm_P7.50mm" (at 47.9552 95.25 0)
+    (property "Footprint" "Capacitor_SMD:C_1812_4532Metric" (at 47.9552 95.25 0)
       (effects (font (size 1.27 1.27)) hide)
     )
@@
       (effects (font (size 1.27 1.27)))
     )
-    (property "Footprint" "Resistor_THT:R_Axial_DIN0207_L6.3mm_D2.5mm_P10.16mm_Horizontal" (at 61.214 63.754 90)
+    (property "Footprint" "Resistor_SMD:R_0805_2012Metric" (at 61.214 63.754 90)
       (effects (font (size 1.27 1.27)) hide)
     )
@@
       (effects (font (size 1.27 1.27)))
     )
-    (property "Footprint" "Diode_THT:D_DO-35_SOD27_P7.62mm_Horizontal" (at 226.06 95.25 0)
+    (property "Footprint" "Diode_SMD:D_2010_5025Metric" (at 226.06 95.25 0)
       (effects (font (size 1.27 1.27)) hide)
     )
@@
       (effects (font (size 1.27 1.27)) (justify right))
     )
-    (property "Footprint" "Resistor_THT:R_Axial_DIN0207_L6.3mm_D2.5mm_P10.16mm_Horizontal" (at 58.674 96.266 90)
+    (property "Footprint" "Resistor_SMD:R_0805_2012Metric" (at 58.674 96.266 90)
       (effects (font (size 1.27 1.27)) hide)
     )
@@
       (effects (font (size 1.27 1.27)))
     )
-    (property "Footprint" "Resistor_THT:R_Axial_DIN0207_L6.3mm_D2.5mm_P10.16mm_Horizontal" (at 215.646 59.436 90)
+    (property "Footprint" "Resistor_SMD:R_0805_2012Metric" (at 215.646 59.436 90)
       (effects (font (size 1.27 1.27)) hide)
     )
@@
       (effects (font (size 1.27 1.27)) (justify right))
     )
-    (property "Footprint" "Resistor_THT:R_Axial_DIN0207_L6.3mm_D2.5mm_P10.16mm_Horizontal" (at 202.184 63.246 90)
+    (property "Footprint" "Resistor_SMD:R_0805_2012Metric" (at 202.184 63.246 90)
       (effects (font (size 1.27 1.27)) hide)
     )
@@
       (effects (font (size 1.27 1.27)) (justify left))
     )
-    (property "Footprint" "Resistor_THT:R_Axial_DIN0207_L6.3mm_D2.5mm_P10.16mm_Horizontal" (at 131.826 100.584 90)
+    (property "Footprint" "Resistor_SMD:R_0805_2012Metric" (at 131.826 100.584 90)
       (effects (font (size 1.27 1.27)) hide)
     )
@@
       (effects (font (size 1.27 1.27)) (justify right))
     )
-    (property "Footprint" "Resistor_THT:R_Axial_DIN0207_L6.3mm_D2.5mm_P10.16mm_Horizontal" (at 166.624 102.616 90)
+    (property "Footprint" "Resistor_SMD:R_0805_2012Metric" (at 166.624 102.616 90)
       (effects (font (size 1.27 1.27)) hide)
     )
@@
       (effects (font (size 1.27 1.27)))
     )
-    (property "Footprint" "Capacitor_THT:CP_Radial_D10.0mm_P3.80mm" (at 133.35 96.2152 0)
+    (property "Footprint" "Capacitor_THT:CP_Radial_D5.0mm_P2.50mm" (at 133.35 96.2152 0)
       (effects (font (size 1.27 1.27)) hide)
     )
@@
       (effects (font (size 1.27 1.27)) (justify left))
     )
-    (property "Footprint" "Capacitor_THT:C_Disc_D11.0mm_W5.0mm_P7.50mm" (at 157.1752 106.68 0)
+    (property "Footprint" "Capacitor_SMD:C_0805_2012Metric" (at 157.1752 106.68 0)
       (effects (font (size 1.27 1.27)) hide)
     )
@@
       (effects (font (size 1.27 1.27)) (justify left))
     )
-    (property "Footprint" "Resistor_THT:R_Axial_DIN0207_L6.3mm_D2.5mm_P10.16mm_Horizontal" (at 36.576 92.964 90)
+    (property "Footprint" "Resistor_SMD:R_0805_2012Metric" (at 36.576 92.964 90)
       (effects (font (size 1.27 1.27)) hide)
     )
@@
       (effects (font (size 1.27 1.27)))
     )
-    (property "Footprint" "Resistor_THT:R_Axial_DIN0207_L6.3mm_D2.5mm_P10.16mm_Horizontal" (at 84.836 75.946 90)
+    (property "Footprint" "Resistor_SMD:R_0805_2012Metric" (at 84.836 75.946 90)
       (effects (font (size 1.27 1.27)) hide)
     )
@@
       (effects (font (size 1.27 1.27)) (justify left))
     )
-    (property "Footprint" "Resistor_THT:R_Axial_DIN0207_L6.3mm_D2.5mm_P10.16mm_Horizontal" (at 260.096 85.344 90)
+    (property "Footprint" "Resistor_SMD:R_0805_2012Metric" (at 260.096 85.344 90)
       (effects (font (size 1.27 1.27)) hide)
     )
@@
       (effects (font (size 1.27 1.27)) (justify left))
     )
-    (property "Footprint" "Capacitor_THT:C_Disc_D11.0mm_W5.0mm_P7.50mm" (at 122.8852 102.87 0)
+    (property "Footprint" "Capacitor_SMD:C_0805_2012Metric" (at 122.8852 102.87 0)
       (effects (font (size 1.27 1.27)) hide)
     )
@@
       (effects (font (size 1.27 1.27)) (justify right))
     )
-    (property "Footprint" "Diode_THT:D_DO-35_SOD27_P7.62mm_Horizontal" (at 27.94 90.17 0)
+    (property "Footprint" "Diode_SMD:D_2010_5025Metric" (at 27.94 90.17 0)
       (effects (font (size 1.27 1.27)) hide)
     )
@@
       (effects (font (size 1.27 1.27)))
     )
-    (property "Footprint" "Resistor_THT:R_Axial_DIN0207_L6.3mm_D2.5mm_P10.16mm_Horizontal" (at 214.376 96.266 90)
+    (property "Footprint" "Resistor_SMD:R_0805_2012Metric" (at 214.376 96.266 90)
       (effects (font (size 1.27 1.27)) hide)
     )
@@
       (effects (font (size 1.27 1.27)) (justify left))
     )
-    (property "Footprint" "Resistor_THT:R_Axial_DIN0207_L6.3mm_D2.5mm_P10.16mm_Horizontal" (at 102.616 109.474 90)
+    (property "Footprint" "Resistor_SMD:R_0805_2012Metric" (at 102.616 109.474 90)
       (effects (font (size 1.27 1.27)) hide)
     )
@@
       (effects (font (size 1.27 1.27)) (justify left))
     )
-    (property "Footprint" "Resistor_THT:R_Axial_DIN0207_L6.3mm_D2.5mm_P10.16mm_Horizontal" (at 36.576 80.264 90)
+    (property "Footprint" "Resistor_SMD:R_0805_2012Metric" (at 36.576 80.264 90)
       (effects (font (size 1.27 1.27)) hide)
     )
@@
       (effects (font (size 1.27 1.27)))
     )
-    (property "Footprint" "Capacitor_THT:C_Disc_D11.0mm_W5.0mm_P7.50mm" (at 217.17 84.1248 0)
-      (effects (font (size 1.27 1.27)) hide)
-    )
+    (property "Footprint" "Capacitor_SMD:C_1812_4532Metric" (at 217.17 84.1248 0)
+      (effects (font (size 1.27 1.27)) hide)
+    )
