File: theremin_smd.kicad_pcb (KiCad board)
At the start: 2 copper layers, 139.7 x 38.1 mm, 108 parts, among them J1 Audio Out, J2 12VAC, Q1 2N3904, Q2 2N3904, Q3 2N3904, Q4 2N3904, Q5 2N3904, Q6 2N3904, Q7 2N3904, Q8 2N3904, SW1 SW_SPDT, U1 LM13600, U2 L7812, U3 L7912

Commit message: Finished VPO
Parts:
- C1, C12, C14, C15, C16, C2, C24, C26, C3, C5, C6, C7, C9: footprint Capacitor_THT:C_Disc_D3.0mm_W1.6mm_P2.50mm -> Capacitor_SMD:C_0805_2012Metric
- C21, C22, C23, C27: footprint Capacitor_THT:C_Disc_D3.8mm_W2.6mm_P2.50mm -> Capacitor_SMD:C_1812_4532Metric
- D1, D2, D3, D4, D5: footprint Diode_THT:D_DO-35_SOD27_P7.62mm_Horizontal -> Diode_SMD:D_2010_5025Metric
- L1, L10, L11, L2, L3, L4, L5, L6, L7, L8, L9: footprint Inductor_THT:L_Axial_L5.3mm_D2.2mm_P7.62mm_Horizontal_Vishay_IM-1 -> Inductor_SMD:L_1210_3225Metric
- R1, R10, R11, R12, R13, R14, R15, R16, R17, R18, R19, R2, R20, R21, R22, R23, R24, R25, R26, R27, R28, R29, R3, R30, R31, R32, R33, R34, R35, R36, R37, R38, R39, R4, R40, R41, R5, R6, R7, R8, R9: footprint Resistor_THT:R_Axial_DIN0204_L3.6mm_D1.6mm_P5.08mm_Horizontal -> Resistor_SMD:R_0805_2012Metric
- moved REF** 14.9 mm to (40.9, 43.4)
- moved C9 6.51 mm to (84.5, 29.2)
- moved R6 6.30 mm to (80.3, 38.8)
- moved R5 5.66 mm to (71.8, 38.1)
- moved R17 5.54 mm to (41.9, 38.4), turned to 0 degrees
- moved R12 5.16 mm to (87.0, 41.3), turned to 180 degrees
- moved C8 5.12 mm to (75.6, 40.1)
- moved C14 4.91 mm to (52.1, 34.6), turned to -90 degrees
- moved R13 4.80 mm to (85.1, 38.7), turned to 0 degrees
- moved R18 4.73 mm to (65.7, 41.6)
- moved R39 4.72 mm to (88.5, 38.7)
- moved C5 4.70 mm to (78.1, 29.2), turned to 90 degrees
- moved Q5 4.60 mm to (89.5, 28.2)
- moved R7 3.83 mm to (80.4, 32.4)
- moved C7 3.83 mm to (81.3, 29.2)
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Routing:
- net Volume Tuning: track 31.5 -> 0.00 mm
- net Volume Antenna B: track 26.7 -> 5.13 mm
- net Net-(Q5-E): track 0.00 -> 19.1 mm, vias 0 -> 1
- net -12V: track 30.7 -> 47.7 mm, vias 0 -> 2
- net +12V: track 88.7 -> 98.9 mm
- net Net-(Q3-C): track 29.6 -> 20.9 mm
- net Net-(C10-Pad1): track 0.00 -> 8.61 mm
- net Net-(Q3-E): track 0.00 -> 8.44 mm
- net Net-(Q6-C): track 17.1 -> 23.9 mm
- net Net-(L10-Pad1): track 0.00 -> 6.24 mm
- net Net-(Q4-B): track 0.00 -> 6.19 mm
- net Net-(Q5-B): track 0.00 -> 5.11 mm
- net Net-(Q3-B): track 0.00 -> 4.19 mm
- net Net-(C7-Pad2): track 7.03 -> 3.05 mm
- net Net-(Q7-B): track 10.7 -> 7.31 mm
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